Commit message: added camera to urfd

File: robots/panda_arm_hand.urdf.xacro (robot description, xacro)
@@ -4,8 +4,15 @@
   <xacro:arg name="load_gripper" default="true"/>
   <xacro:arg name="load_gazebo" default="false"/>
+  <xacro:arg name="load_camera" default="true" />
   <xacro:include filename="$(find franka_panda_description)/robots/panda_arm.xacro"/>
   <xacro:if value="$(arg load_gripper)">
-    <xacro:include filename="$(find franka_panda_description)/robots/hand.xacro"/>
-    <xacro:hand ns="panda" rpy="0 0 ${-pi/4}" connected_to="panda_link8"/>
+     <xacro:include filename="$(find franka_panda_description)/robots/hand.xacro"/>
+     <xacro:hand ns="panda" rpy="0 0 ${-pi/4}" connected_to="panda_link8"/>
+  </xacro:if>
+   <xacro:if value="$(arg load_camera)">
+      <xacro:include filename="$(find realsense2_description)/urdf/_d435.urdf.xacro" />
+    <xacro:sensor_d435 name="rgbd" parent="$(arg robot_name)_hand">
+        <origin xyz="0.02 0.0 0.02" rpy="0.0 0.0 0.0" />
+    </xacro:sensor_d435>
   </xacro:if>
   <xacro:if value="$(arg load_gazebo)">
